File: TSOC_GROVEY_FOUR/TSOC_GROVEY_FOUR.sch (EAGLE design)
At the start: 38 parts, among them J2 JTAG-ISSPMIN, J3 4P-2.0-90D, J4 4P-2.0-90D, J5 4P-2.0-90D, J6 4P-2.0-90D, U1 CY8C4XXX-28

Commit message: update Rev 3.0
Parts:
- removed D1: (no value), TSOC-ESP8266-BASE:LED0603
- removed J2: JTAG-ISSPMIN, PatternAgents-Cypress:JTAG-ISSPMIN
- removed J3, J4, J5, J6: 4P-2.0-90D, Seeed-Connector -2016:GROVE-CONNECTOR-DIP-90D(4P-2.0)
- removed U$101: TSOC-LOGO-LRG, thingSoC:TSOC-LOGO-LRG
- removed U$3: TSOC-24-BB, thingSoC:TSOC-24-BB
- added 5V0, GND: (no value), PatternAgents-ProtoPads:M01PTH
- added AIO, DIO, I2C, UART: 4P-2.0-90D, Seeed-Connector -2016:GROVE-CONNECTOR-DIP-90D(4P-2.0)
- added C11, C15, C16, C17: 100nf, Seeed-Capacitor-2016:CERAMIC-100NF-50V-10%-X7R(0603)
- added C12, C14: 1uF, Seeed-Capacitor-2016:CERAMIC-100NF-50V-10%-X7R(0603)
- added C13: 22uF, TSOC_USBUART2:CAP-1206
- added FTDI: 6p-2.54, Seeed-Connector -2016:DIP-BLACK-MALE-HEADER(6P-2.54)
- added JTAG: JTAG-ISSPMIN, PatternAgents-Cypress:JTAG-ISSPMIN
- added L1, L2: 120OHM-500MA, Seeed-Inductor-2016:SMD-FERRITE-CHIP-120-OHM-500MA(0603)
- added LED1: GREEN-0603, Seeed-LED-2016:SMD-LED-CLEAR-GREEN(0603)
- added LED2: RED-0603, Seeed-LED-2016:SMD-LED-CLEAR-GREEN(0603)
- added R11: 1K 1/10W, Seeed-Resistor-2016:SMD-RES-1K-5%-1/10W(0603)
- added TSOC: TSOC-24-BB, thingSoC:TSOC-24-BB
- added U$102: TSOC-LOGO-LRG, thingSoC:TSOC-LOGO-LRG
- added U2: CY8C4XXX-28, PatternAgents-Cypress:CY8C4XXX-28
- C1, C4: value 1uF -> 100nf; device SparkFun-Passives:CAP0603-CAP -> Seeed-Capacitor-2016:CERAMIC-100NF-50V-10%-X7R(0603)
- C10: device SparkFun-Passives:CAP0603-CAP -> Seeed-Capacitor-2016:CERAMIC-100NF-50V-10%-X7R(0603)
- C2, C7: value 1uF -> 100nf; device PatternAgents-Misc:CAP0603-CAP -> Seeed-Capacitor-2016:CERAMIC-100NF-50V-10%-X7R(0603)
- C3: value 0.1uF -> 10uf; device PatternAgents-Misc:CAP0603-CAP -> Seeed-Capacitor-2016:CERAMIC-10UF-10V-10%-X5R(0603)
- C5: value 1uF -> 10uf; device PatternAgents-Misc:CAP0603-CAP -> Seeed-Capacitor-2016:CERAMIC-10UF-10V-10%-X5R(0603)
- C6: value 0.1uF -> 470Pf; device PatternAgents-Misc:CAP0603-CAP -> Seeed-Capacitor-2016:CERAMIC-100NF-50V-10%-X7R(0603)
- C8: value 0.1uF -> 2.2nf; device PatternAgents-Misc:CAP0603-CAP -> Seeed-Capacitor-2016:CERAMIC-1NF-50V-5%-C0G(0603)
- C9: value 1uF -> 10nf; device SparkFun-Passives:CAP0603-CAP -> Seeed-Capacitor-2016:CERAMIC-10NF-50V-10%-X7R(0603)
- J1: value (none) -> NO
- R1: value 2k2 -> 1K 1/10W; device SparkFun-Passives:RESISTOR0603-RES -> Seeed-Resistor-2016:SMD-RES-1K-5%-1/10W(0603)
- R10: device PatternAgents-Misc:RESISTOR_SFE0603-RES -> Seeed-Resistor-2016:SMD-RES-2.2K-5%-1/10W(0603)
- R2: value 10K -> 2.2K; device PatternAgents-Misc:RESISTOR_SFE0603-RES -> Seeed-Resistor-2016:SMD-RES-2.2K-5%-1/10W(0603)
- R3: value 2k2 -> 2.2K; device SparkFun-Passives:RESISTOR0603-RES -> Seeed-Resistor-2016:SMD-RES-2.2K-5%-1/10W(0603)
- R4, R5, R8, R9: value 2k2 -> 1K; device SparkFun-Passives:RESISTOR0603-RES -> Seeed-Resistor-2016:SMD-RES-2.2K-5%-1/10W(0603)
- R6: value DNP -> 10K 1/10W; device SparkFun-Passives:RESISTOR0603-RES -> Seeed-Resistor-2016:SMD-RES-10K-5%-1/10W(0603)
- R7: value DNP -> 1K; device SparkFun-Passives:RESISTOR0603-RES -> Seeed-Resistor-2016:SMD-RES-2.2K-5%-1/10W(0603)
- U$1: value TSOC-LOGO-MED -> TSOC-LOGO-SMALL; device thingSoC:TSOC-LOGO-MED -> thingSoC:TSOC-LOGO-SMALL
- U$4: value TSOC-LOGO-MED -> TSOC-LOGO; device thingSoC:TSOC-LOGO-MED -> thingSoC:TSOC-LOGO
- U1: value CY8C4XXX-28 -> MIC5219 3.3V; device PatternAgents-Cypress:CY8C4XXX-28 -> TSOC-ESP8266-BASE:V_REG_MIC52193.3V
- renumbered U$100 to U$103, U$2 to $$U$1
Connections:
- new net !URST: C7.1, FTDI.6
- new net BYPASS1: C6.1, U1.BP
- new net LEDR: LED2.-, R11.1
- new net P0_6E: AIO.2, R7.2
- new net P0_7E: AIO.1, R8.2
- new net P1_0E: DIO.1, R10.2
- new net P1_1E: DIO.2, R9.2
- new net P4_0E: R5.2, UART.2
- new net P4_1E: R4.2, UART.1
- new net TSOC_3V3: L2.2, TSOC.3V3
- new net TSOC_5V0: L1.2, TSOC.5V0
- net !XRES: now also C7.2, JTAG.3, R6.1, U2.!XRES; no longer J2.3, R2.1, U$3.!ATN, U1.!XRES
- net 3V3: now also C5.2, L2.1, U1.OUT; no longer U$3.3V3
- net 5V0: now also 5V0.1, C3.2, C4.1, L1.1, U1.EN, U1.IN; no longer U$3.5V0
- net GND: now also AIO.4, C10.1, C11.1, C12.1, C13.2, C14.1, C15.1, C16.2, C17.2, C3.1, C5.1, C8.1, C9.1, DIO.4, FTDI.1, FTDI.2, GND.1, I2C.4, JTAG.2, LED1.-, TSOC.AGND, TSOC.GND, U1.GND, U2.VSS, UART.4; no longer C10.2, C3.2, C5.2, C7.2, C8.2, C9.2, D1.C, J2.2, J3.4, J4.4, J5.4, J6.4, U$3.AGND, U$3.GND, U1.VSS
- net N$17: now also LED1.+, R1.1; no longer D1.A, R10.1
- net P0_0: now also TSOC.!CTS, U2.P0_0; no longer U$3.SS1, U1.P0_0
- net P0_1: now also TSOC.!RTS, U2.P0_1; no longer U$3.SS2, U1.P0_1
- net P0_2: now also TSOC.!DTR, U2.P0_2; no longer U$3.!CS, U1.P0_2
- net P0_3: now also TSOC.!DSR, U2.P0_3; no longer R10.2, U$3.SCK, U1.P0_3
- net P0_6: now also R7.1, TSOC.!DCD, U2.P0_6; no longer U$3.MISO, U1.P0_7
- net P0_7: now also R8.1, TSOC.!RI, U2.P0_7; no longer U$3.MOSI, U1.P0_6
- net P1_0: now also R10.1, TSOC.IO2, U2.P1_0; no longer U$3.RXD, U1.P1_0
- net P1_1: now also R9.1, TSOC.IO1, U2.P1_1; no longer U$3.TXD, U1.P1_1
- net P1_2: now also R11.2, TSOC.SS2, U2.P1_2; no longer U$3.!CTS, U1.P1_2
- net P1_7: now also C11.2, C12.2, TSOC.SS1, U2.P1_7; no longer C2.1, C3.1, U1.P1_7
- net P2_2: now also TSOC.!IRQ, U2.P2_2; no longer U$3.!RTS, U1.P2_2
- net P2_3: now also TSOC.!ATN, U2.P2_3; no longer U$3.!DTR, U1.P2_3
- net P2_4: now also TSOC.!CS, U2.P2_4; no longer J6.2, R8.1, U$3.!DSR, U1.P2_4
- net P2_5: now also TSOC.SCK, U2.P2_5; no longer J6.1, R9.1, U$3.!DCD, U1.P2_5
- net P2_6: now also TSOC.MISO, U2.P2_6; no longer J4.2, R4.1, U$3.!RI, U1.P2_6
- net P2_7: now also TSOC.MOSI, U2.P2_7; no longer J4.1, R5.1, U$3.!IRQ, U1.P2_7
- net P3_0: now also I2C.1, R2.1, TSOC.SCL, U2.P3_0; no longer J3.1, R1.1, U$3.SCL, U1.P3_0
- net P3_1: now also I2C.2, TSOC.SDA, U2.P3_1; no longer J3.2, U$3.SDA, U1.P3_1
- net P3_2: now also JTAG.5, U2.P3_2; no longer J2.5, U1.P3_2
- net P3_3: now also JTAG.4, U2.P3_3; no longer J2.4, U1.P3_3
- net P4_0: now also FTDI.4, R5.1, TSOC.RXD, U2.P4_0; no longer J5.2, R7.1, U1.P4_0
- net P4_1: now also FTDI.5, R4.1, TSOC.TXD, U2.P4_1; no longer J5.1, R6.1, U1.P4_1
- net P4_2: now also C8.2, U2.P4_2; no longer U$3.IO2, U1.P4_2
- net P4_3: now also C9.2, U2.P4_3; no longer U$3.IO1, U1.P4_3
- net VCC: now also AIO.3, C13.1, C14.2, C15.2, C16.1, C17.1, C2.1, DIO.3, FTDI.3, I2C.3, JTAG.1, LED2.+, U2.VDDD, UART.3; no longer C10.1, C4.1, C5.1, C6.1, C9.1, J2.1, J3.3, J4.3, J5.3, J6.3, R4.2, R5.2, R7.2, R8.2, R9.2, U1.VDDD
- net VCCD: now also C10.2, U2.VCCD; no longer C7.1, C8.1, U1.VCCD
Other:
- note added: "3.3V LDO/Regulator"
- note added: "AIN"
- note added: "CapSense Tank"
- note added: "FTDI UART"
- note removed: "DNP"
- note removed: "Notes: 1) Add GND Looper 2) Add TP for JTAG 3) Change UART to UARTM (master)"
- note removed: "SIG1"
- note removed: "SIG2"
- note removed: "SIG3"
- note removed: "SIG4"
- moved on the sheet: J1
