File: TSOC_GROVEY_FOUR/TSOC_GROVEY_FOUR.sch (EAGLE design)
At the start: 53 parts, among them J1 NO, U1 XC6204B332MR-SOT23-5, U2 CY8C4XXX-28

Commit message: update to Rev3.1
Parts:
- removed U$103: TSOC-LOGO-SMALL, thingSoC:TSOC-LOGO-SMALL
- added R12, R13: 1K 1/10W, Seeed-Resistor-2016:SMD-RES-1K-5%-1/10W(0603)
- added U$101: TSOC-LOGO-LRG, thingSoC:TSOC-LOGO-LRG
- C6: value 1nf -> 100nf; device Seeed-Capacitor-2016:CERAMIC-1NF-50V-10%-X7R(0603) -> Seeed-Capacitor-2016:CERAMIC-100NF-50V-10%-X7R(0603)
- R2, R3: value 2.2K -> 1K 1/10W; device Seeed-Resistor-2016:SMD-RES-2.2K-5%-1/10W(0603) -> Seeed-Resistor-2016:SMD-RES-1K-5%-1/10W(0603)
- R7, R8: value 1K 1/10W -> 10K 1/10W; device Seeed-Resistor-2016:SMD-RES-1K-5%-1/10W(0603) -> Seeed-Resistor-2016:SMD-RES-10K-5%-1/10W(0603)
- U$102: value TSOC-LOGO-LRG -> TSOC-LOGO-SMALL; device thingSoC:TSOC-LOGO-LRG -> thingSoC:TSOC-LOGO-SMALL
- U1: value XC6204B332MR-SOT23-5 -> 3.3V; device Seeed-IC-2016:PMIC-LDO-XC6204B332MR(SOT23-5) -> SparkFun-PowerIC:V_REG_AP2112K-3.3V
- renumbered AIO to J4, DIO to J5, I2C to J2, UART to J3
Connections:
- net BYPASS1 renamed N$1
- net N$17 renamed LED1
- net P4_0E renamed D2
- net P4_1E renamed A2
- removed net LEDR: LED2.-, R11.1
- removed net P0_6E: J4.2, R7.2
- removed net P0_7E: J4.1, R8.2
- removed net P1_0E: J5.1, R10.2
- removed net P1_1E: J5.2, R9.2
- new net A1: J2.1, R2.2
- new net A3: J4.1, R10.2
- new net A4: J5.1, R12.2
- new net D1: J2.2, R3.2
- new net D3: J4.2, R9.2
- new net D4: J5.2, R11.2
- new net LED2: LED2.-, R13.1
- net !XRES: now also R7.1; no longer R6.1
- net 3V3: now also U1.OUT; no longer U1.VOUT
- net 5V0: now also U1.EN, U1.IN; no longer U1.CE, U1.VIN
- net GND: now also U1.GND; no longer U1.VSS
- net P0_0: now also R3.1
- net P0_6: no longer R7.1
- net P0_7: no longer R8.1
- net P1_0: now also R9.1; no longer R10.1, TSOC.IO2
- net P1_1: now also R5.1; no longer R9.1, TSOC.IO1
- net P1_2: now also R11.1, R13.2; no longer R11.2, TSOC.SS2
- net P1_7: no longer TSOC.SS1
- net P2_4: now also R10.1; no longer TSOC.!CS
- net P2_5: now also R12.1; no longer TSOC.SCK
- net P2_6: now also R4.1; no longer TSOC.MISO
- net P2_7: now also R2.1; no longer TSOC.MOSI
- net P3_0: now also R8.1; no longer J2.1, R2.1
- net P3_1: now also R6.1; no longer J2.2, R3.1
- net P4_0: now also TSOC.TXD; no longer R5.1, TSOC.RXD
- net P4_1: now also TSOC.RXD; no longer R4.1, TSOC.TXD
- net VCC: now also R7.2, R8.2; no longer R2.2, R3.2
Other:
- note added: "ANALOG"
- note added: "DOUT"
- note added: "Rev 3.1 Notes: 1) Move P2_3 (ADC) to AIO 2) Swap UART TX/RX to match GroveyOne 3) Change U1 to CJ1117B"
- note added: "SLAVE"
- note removed: "RXD"
- note removed: "SCL"
- note removed: "SDA"
- note removed: "TXD"
- moved on the sheet: C6, R10, R11, R2, R3, R6, R7, R8, R9
