File: TSOC_GROVEY_FOUR/revisions/R3_0/TSOC_GROVEY_FOUR.sch (EAGLE design)
At the start: 50 parts, among them J1 4P-2.0-90D, J2 4P-2.0-90D, J3 NO, J4 6p-2.54, J5 4P-2.0-90D, J6 4P-2.0-90D, J7 JTAG-ISSPMIN, U1 MIC5219 3.3V, U2 CY8C4XXX-28

Commit message: update Rev 3.0
Parts:
- removed J2: 4P-2.0-90D, Seeed-Connector -2016:GROVE-CONNECTOR-DIP-90D(4P-2.0)
- removed J3: NO, PatternAgents-ProtoPads:JMP-3-NO-PTH
- removed U$101: TSOC-LOGO-SMALL, thingSoC:TSOC-LOGO-SMALL
- added 5V0: (no value), PatternAgents-ProtoPads:M01PTH
- added C16, C17: 100nf, Seeed-Capacitor-2016:CERAMIC-100NF-50V-10%-X7R(0603)
- added I2C, UART: 4P-2.0-90D, Seeed-Connector -2016:GROVE-CONNECTOR-DIP-90D(4P-2.0)
- added U$4: TSOC-LOGO, thingSoC:TSOC-LOGO
- C10, C12: value 100nf -> 1uF
- C11: value 22uF -> 100nf; device TSOC_USBUART2:CAP-1206 -> Seeed-Capacitor-2016:CERAMIC-100NF-50V-10%-X7R(0603)
- C13: value 100nf -> 22uF; device Seeed-Capacitor-2016:CERAMIC-100NF-50V-10%-X7R(0603) -> TSOC_USBUART2:CAP-1206
- C15, C7: value 1uF -> 100nf
- C6: value 100nf -> 470Pf
- C8: value 470Pf -> 2.2nf; device Seeed-Capacitor-2016:CERAMIC-100NF-50V-10%-X7R(0603) -> Seeed-Capacitor-2016:CERAMIC-1NF-50V-5%-C0G(0603)
- C9: value 100nf -> 10nf; device Seeed-Capacitor-2016:CERAMIC-100NF-50V-10%-X7R(0603) -> Seeed-Capacitor-2016:CERAMIC-10NF-50V-10%-X7R(0603)
- J1: value 4P-2.0-90D -> NO; device Seeed-Connector -2016:GROVE-CONNECTOR-DIP-90D(4P-2.0) -> PatternAgents-ProtoPads:JMP-3-NO-PTH
- R10, R4, R5, R7, R8, R9: value 2.2K -> 1K
- renumbered J4 to FTDI, J5 to AIO, J6 to DIO, J7 to JTAG
Connections:
- removed net $1: TSOC.SS1, TSOC.SS2
- new net P0_6E: AIO.2, R7.2
- new net P0_7E: AIO.1, R8.2
- new net P1_0E: DIO.1, R10.2
- new net P1_1E: DIO.2, R9.2
- new net P4_0E: R5.2, UART.2
- new net P4_1E: R4.2, UART.1
- net !URST: now also C7.1; no longer C9.1
- net !XRES: now also C7.2; no longer C9.2
- net 3V3: now also J1.1; no longer J3.1
- net 5V0: now also 5V0.1, J1.3; no longer J3.3
- net BYPASS1: now also C6.1; no longer C8.1
- net GND: now also C11.1, C12.1, C16.2, C17.2, C6.2, C8.1, C9.1, I2C.4, UART.4; no longer C11.2, C12.2, C6.1, C7.1, C8.2, J1.4, J2.4
- net P0_2: no longer AIO.2, R7.1
- net P0_3: no longer J1.1, R11.2, R4.1
- net P0_6: now also R7.1, TSOC.!DCD, U2.P0_6; no longer TSOC.!RI, U2.P0_7
- net P0_7: now also R8.1, TSOC.!RI, U2.P0_7; no longer J1.2, R5.1, TSOC.!DCD, U2.P0_6
- net P1_0: now also R10.1
- net P1_1: now also R9.1
- net P1_2: now also R11.2, TSOC.SS2
- net P1_7: now also C11.2, C12.2, TSOC.SS1; no longer C15.2, C6.2
- net P2_4: no longer AIO.1, R8.1
- net P2_6: no longer DIO.1, R10.1
- net P3_0: now also I2C.1; no longer J2.1
- net P3_1: now also I2C.2; no longer J2.2
- net P4_0: now also R5.1
- net P4_1: now also R4.1
- net P4_2: now also C8.2; no longer DIO.2, R9.1
- net P4_3: now also C9.2
- net VCC: now also C15.2, C16.1, C17.1, I2C.3, J1.2, UART.3; no longer C10.2, C11.1, C12.1, J1.3, J2.3, J3.2, R10.2, R4.2, R5.2, R7.2, R8.2, R9.2
- net VCCD: now also C10.2; no longer C7.2
Other:
- note added: "AIN"
- note added: "CapSense Tank"
- note added: "FTDI UART"
- moved on the sheet: C1, C10, C12, C15, C2, C6, C7, C8, C9, R10, R2, R3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
