File: TSOC_GROVEY_FOUR/revisions/R3_1/TSOC_GROVEY_FOUR.brd (EAGLE design)
At the start: 44.5 x 30.5 mm, 57 parts, among them J1 NO, U1 XC6204B332MR-SOT23-5, U2 CY8C4XXX-28

Commit message: update Rev 3.0
Parts:
- removed C6: 1nf, Seeed-Capacitor-2016:C0603
- U1: value XC6204B332MR-SOT23-5 -> CJA1117B-3.3-SOT89; device Seeed-IC-2016:SOT-23-5 -> Seeed-IC-2016:SOT-89
- moved U1 1.37 mm to (14.5, 17.0), turned to 270 degrees
Connections:
- net LEDR renamed LED2
- net N$17 renamed LED1
- removed net BYPASS1: C6.1, U1.4
- net 3V3: now also U1.2, U1.4; no longer U1.5
- net 5V0: no longer U1.1
- net GND: now also U1.1; no longer C6.2, U1.2
- net P0_7: no longer R8.1
- net P2_3: now also R8.1
- net P4_0: now also R4.1, TSOC.8C; no longer R5.1, TSOC.7C
- net P4_0E: now also R4.2, UART.1; no longer R5.2, UART.2
- net P4_1: now also R5.1, TSOC.7C; no longer R4.1, TSOC.8C
- net P4_1E: now also R5.2, UART.2; no longer R4.2, UART.1
Routing:
- net P2_3: track 7.93 -> 22.5 mm, vias 0 -> 2
- net P0_7: track 24.9 -> 17.8 mm, vias 2 -> 1
- net P0_6: track 23.9 -> 30.9 mm
- net P3_3: track 14.4 -> 21.0 mm, vias 2 -> 1
- net P4_0: track 35.6 -> 40.2 mm
- net P3_2: track 10.4 -> 14.3 mm
- net 5V0: track 38.9 -> 35.3 mm
- net 3V3: track 33.9 -> 37.4 mm
- net GND: track 213.2 -> 216.2 mm
- net P4_1: track 31.8 -> 34.2 mm
- net BYPASS1: track 2.26 -> 0.00 mm
- net P2_5: track 10.1 -> 11.1 mm
- net P3_0: track 34.9 -> 35.7 mm
- net P2_7: track 13.6 -> 14.3 mm
- net !XRES: track 35.0 -> 34.4 mm
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Other:
- board text added: "Rev. 3.1"
- board text removed: "Rev. 3.0"
- board text removed: "by"

Commit message: update to Rev3.1
Parts:
- removed U$103: TSOC-LOGO-SMALL, thingSoC:TSOC-LOGO-SML
- added C6: 100nf, Seeed-Capacitor-2016:C0603
- added R12, R13: 1K 1/10W, Seeed-Resistor-2016:R0603
- added U$101: TSOC-LOGO-LRG, thingSoC:TSOC-LOGO-LRG
- R2, R3: value 2.2K -> 1K 1/10W
- R7, R8: value 1K 1/10W -> 10K 1/10W
- U$102: value TSOC-LOGO-LRG -> TSOC-LOGO-SMALL; device thingSoC:TSOC-LOGO-LRG -> thingSoC:TSOC-LOGO-SML
- U1: value CJA1117B-3.3-SOT89 -> 3.3V; device Seeed-IC-2016:SOT-89 -> SparkFun-PowerIC:SOT23-5
- moved R7 17.4 mm to (17.0, 8.13), turned to 0 degrees
- moved R8 17.0 mm to (17.3, 13.0), turned to 0 degrees
- moved U$102 11.4 mm to (42.4, 14.5)
- moved R9 10.4 mm to (34.3, 10.2)
- moved R10 10.4 mm to (34.3, 13.2), turned to 180 degrees
- moved R11 8.85 mm to (34.3, 20.6), turned to 180 degrees
- moved R6 6.10 mm to (15.5, 13.0)
- moved C7 1.80 mm to (18.5, 8.13)
- moved U$3 1.37 mm to (1.02, 24.1)
- moved U1 1.37 mm to (13.2, 16.5), turned to 0 degrees
- moved $$U$3 1.30 mm to (40.1, 24.1)
- moved U$100 1.30 mm to (5.59, 15.5)
- moved $$U$2 0.92 mm to (39.9, 13.5)
- moved U$1 0.92 mm to (1.02, 13.5)
- renumbered AIO to J4, DIO to J5, I2C to J2, UART to J3
Connections:
- net P4_0E renamed A2
- net P4_1E renamed D2
- removed net P0_6E: J4.2, R7.2
- removed net P0_7E: J4.1, R8.2
- removed net P1_0E: J5.1, R10.2
- removed net P1_1E: J5.2, R9.2
- new net A1: J2.1, R2.2
- new net A3: J4.1, R10.2
- new net A4: J5.1, R12.2
- new net D1: J2.2, R3.2
- new net D3: J4.2, R9.2
- new net D4: J5.2, R11.2
- new net N$1: C6.1, U1.4
- net !XRES: now also R7.1; no longer R6.1
- net 3V3: now also U1.5; no longer U1.2, U1.4
- net 5V0: now also U1.1
- net GND: now also C6.2, U1.2; no longer U1.1
- net LED2: now also R13.1; no longer R11.1
- net P0_0: now also R3.1
- net P0_6: no longer R7.1
- net P1_0: now also R9.1; no longer R10.1, TSOC.1B
- net P1_1: now also R5.1; no longer R9.1, TSOC.2B
- net P1_2: now also R11.1, R13.2; no longer R11.2, TSOC.3B
- net P1_7: no longer TSOC.4B
- net P2_3: no longer R8.1
- net P2_4: now also R10.1; no longer TSOC.7B
- net P2_5: now also R12.1; no longer TSOC.8B
- net P2_6: now also R4.1; no longer TSOC.9B
- net P2_7: now also R2.1; no longer TSOC.10B
- net P3_0: now also R8.1; no longer J2.1, R2.1
- net P3_1: now also R6.1; no longer J2.2, R3.1
- net P4_0: no longer R4.1
- net P4_1: no longer R5.1
- net VCC: now also R7.2, R8.2; no longer R2.2, R3.2
Routing:
- net P4_1: track 34.2 -> 11.6 mm, vias 2 -> 0
- net P4_0: track 40.2 -> 18.2 mm, vias 3 -> 1
- net P0_0: track 9.28 -> 27.0 mm, vias 0 -> 2
- net P0_6: track 30.9 -> 13.9 mm, vias 1 -> 0
- net P3_0: track 35.7 -> 20.3 mm, vias 3 -> 0
- net P2_3: track 22.5 -> 7.93 mm, vias 2 -> 0
- net P1_2: track 19.4 -> 32.8 mm, vias 0 -> 2
- net P3_1: track 32.0 -> 20.6 mm, vias 3 -> 0
- net P2_7: track 14.3 -> 23.7 mm, vias 1 -> 2
- net P1_7: track 19.6 -> 10.8 mm, vias 1 -> 0
- net P3_3: track 21.0 -> 13.2 mm
- net P2_4: track 8.71 -> 15.9 mm, vias 1 -> 2
- net P1_0: track 15.3 -> 21.8 mm, vias 0 -> 2
- net GND: track 216.2 -> 209.8 mm
- net P2_6: track 12.7 -> 18.7 mm, vias 1 -> 2
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Other:
- board text added: "0_7"
- board text added: "ANALOG"
- board text added: "NC"
- board text added: "P0_0"
- board text added: "P1_2"
- board text added: "P2_4"
- board text added: "P2_5"
- board text added: "P2_6"
- board text added: "P2_7"
- board text removed: "(AREF)"
- board text removed: "(CS0)"
- board text removed: "(LED2)"
- board text removed: "(MISO)"
- board text removed: "(MOSI)"
- board text removed: "(SCK)"
- board text removed: "1_0"
- board text removed: "1_1"
- board text removed: "1_2"
- board text removed: "1_7"
- board text removed: "2_4"
- board text removed: "2_5"
- board text removed: "2_6"
- board text removed: "2_7"
- board text removed: "AIO"
- board text removed: "DIO"
- board text removed: "I2C"
- board text removed: "P0_6"
- board text removed: "P3_0"
- board text removed: "P3_1"
- board text removed: "P4_0"
- board text removed: "P4_1"
